File: PCB/stylophone.brd (EAGLE design)
At the start: 75.3 x 41.2 mm, 25 parts, among them IC2 LM358N

Commit message: w
Connections:
- new net V+: IC2.8
- new net V-: IC2.4
Routing:
- net GND: track 125.0 -> 122.2 mm
Other:
- board text added: "277950"
Changed lines of the file:
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@@
 <circle x="53.2" y="65.2" radius="0.4" width="0.6096" layer="16"/>
 <circle x="11.46" y="53.53" radius="0.4" width="0.6096" layer="16"/>
+<text x="36.8" y="48.4" size="1.778" layer="16" rot="MR0">277950</text>
 </plain>
 <attributes>
@@
 <wire x1="3.41" y1="50.66" x2="3.41" y2="52.61" width="0.6096" layer="16"/>
 <wire x1="3.41" y1="52.61" x2="6" y2="55.2" width="0.6096" layer="16"/>
-<wire x1="6" y1="55.2" x2="6" y2="57.6" width="0.6096" layer="16"/>
-<wire x1="6" y1="57.6" x2="6" y2="60.4" width="0.6096" layer="16"/>
-<wire x1="6" y1="60.4" x2="6" y2="62" width="0.6096" layer="16"/>
+<wire x1="6" y1="55.2" x2="6" y2="62" width="0.6096" layer="16"/>
 <wire x1="6" y1="62" x2="6.8" y2="62.8" width="0.6096" layer="16"/>
 <wire x1="6.89" y1="62.96" x2="21.24" y2="62.96" width="0.6096" layer="16"/>
-<wire x1="6" y1="57.6" x2="3.2" y2="57.6" width="0.6096" layer="16"/>
-<wire x1="6" y1="60.4" x2="3.2" y2="60.4" width="0.6096" layer="16"/>
 <wire x1="6.8" y1="62.8" x2="3.6" y2="62.8" width="0.6096" layer="16"/>
 <wire x1="30.8" y1="53.6" x2="36.8" y2="53.6" width="0.4064" layer="16"/>
@@
 <wire x1="39.6" y1="50.8" x2="41.6" y2="50.8" width="0.4064" layer="16"/>
 <wire x1="41.6" y1="50.8" x2="45.4" y2="54.6" width="0.4064" layer="16"/>
+<wire x1="3.2" y1="60.4" x2="3.2" y2="57.6" width="0.4064" layer="16"/>
 <wire x1="28" y1="50.8" x2="23.88" y2="51.06" width="0" layer="19" extent="16-16"/>
 <wire x1="6.89" y1="62.96" x2="6.8" y2="62.8" width="0" layer="19" extent="16-16"/>
+<wire x1="3.2" y1="60.4" x2="3.6" y2="62.8" width="0" layer="19" extent="16-16"/>
 <wire x1="10.89" y1="62.96" x2="6.89" y2="62.96" width="0" layer="19" extent="16-16"/>
 </signal>
@@
 <wire x1="1.2" y1="47.2" x2="1.2" y2="48" width="0.4064" layer="16"/>
 </signal>
+<signal name="V+">
+<contactref element="IC2" pad="8"/>
+</signal>
+<signal name="V-">
+<contactref element="IC2" pad="4"/>
+</signal>
 </signals>
